Commit message: coche_urdf

File: Paquetes_Ros2/coche_urdf/urdf/qev-3d.urdf.xacro (robot description, xacro)
@@ -7,23 +7,17 @@
   <xacro:property name="degrees_90" value="1.5708"/>
   <xacro:property name="M_PI" value="3.1415926535897931" />
-  <xacro:property name="steering_limit" default="0.28"/>
+  <xacro:property name="steering_limit" default="0.32"/>
   <xacro:property name="wheel_diameter" value="0.4064"/>
+  <xacro:property name="elevacion_coche" value="0.21"/>
   <xacro:property name="wheel_width" value="0.2"/>
-  <xacro:property name="chassis_width" value="1.6"/>
-  <xacro:property name="wheelbase" value="1.580"/>
-  <!-- material -->
-  <material name="black">
-    <color rgba="0 0 0 1"/>
-  </material>
-  <material name="orange">
-    <color rgba="0.88 0.36 0.035 1"/>
-  </material>
+  <xacro:property name="chassis_width" value="1.4"/>
+  <xacro:property name="wheelbase" value="1.5"/>
   <!-- Vehicle include -->
   <xacro:include filename="$(find coche_urdf)/urdf/vehicle.urdf.xacro"/>
   <!-- Chassis of the car -->
   <xacro:chassis base_frame="$(arg base_frame)" display_car="$(arg display_car)"/>
-  <!-- Wheels -->
-  <xacro:wheels/>
-  <!-- Sensors include -->
+  <!-- Wheels
+  <xacro:wheels/>-->
+  <!-- Sensors include
   <xacro:include filename="$(find coche_urdf)/urdf/sensors.urdf.xacro"/>
   <xacro:velodyne parent="${chassis_link}" name="velodyne">
@@ -32,4 +26,4 @@
   <xacro:zed2i parent="${chassis_link}" name="zed2i">
     <origin xyz="-0.370 0.0 0.900" rpy="0 0 0"/>
-  </xacro:zed2i>
+  </xacro:zed2i>-->
 </robot>

File: Paquetes_Ros2/coche_urdf/urdf/sensors.urdf.xacro (robot description, xacro)
@@ -11,10 +11,10 @@
       <visual>
         <geometry>
-          <mesh filename="file://$(find vehicle_urdf)/meshes/VLP16_base_1.dae" />
+          <mesh filename="file://$(find coche_urdf)/meshes/VLP16_base_1.dae" />
         </geometry>
       </visual>
       <visual>
         <geometry>
-          <mesh filename="file://$(find vehicle_urdf)/meshes/VLP16_base_2.dae" />
+          <mesh filename="file://$(find coche_urdf)/meshes/VLP16_base_2.dae" />
         </geometry>
       </visual>
@@ -30,5 +30,5 @@
         <origin xyz="0 0 -0.0377" />
         <geometry>
-          <mesh filename="file://$(find vehicle_urdf)/meshes/VLP16_scan.dae" />
+          <mesh filename="file://$(find coche_urdf)/meshes/VLP16_scan.dae" />
         </geometry>
       </visual>

File: Paquetes_Ros2/coche_urdf/urdf/vehicle.urdf.xacro (robot description, xacro)
@@ -18,5 +18,5 @@
           <origin xyz="0 0 0" rpy="0 0 0"/>
           <geometry>
-            <mesh filename="file://$(find coche_urdf)/meshes/body_06.dae"/>
+            <mesh filename="file://$(find coche_urdf)/meshes/body_x.dae"/>
           </geometry>
         </xacro:if>
@@ -31,6 +31,6 @@
       <origin xyz="0 0 0" rpy="0 0 0"/>
     </link>
-  </xacro:macro>
-  <!-- Wheels -->
+    </xacro:macro>
+    <!-- Wheels -->
   <xacro:macro name="wheels">
     <!-- Wheel description -->
@@ -40,18 +40,15 @@
           <origin xyz="0 0 0" rpy="${degrees_90} 0 0"/>
           <geometry>
-            <cylinder radius="${wheel_diameter / 2}" length="${wheel_width}"/>
+            <mesh filename="file://$(find coche_urdf)/meshes/fr_x.dae"/>
           </geometry>
-          <material name="black"/>
         </visual>
       </link>
     </xacro:macro>
-    <!-- Front and rear wheel descriptions -->
+     <!-- Front and rear wheel descriptions -->
     <!-- Description of how a front wheel is connected to the chassis -->
     <xacro:macro name="front_wheel" params="lr_prefix lr_reflect">
       <link name="${lr_prefix}_steering_hinge"/>
       <joint name="${lr_prefix}_steering_hinge_joint" type="fixed">
-        <origin xyz="${wheelbase / 2}
-                     ${lr_reflect * ((chassis_width - wheel_width) / 2)}
-                     0"
+        <origin xyz="0 0 0"
                 rpy="0 0 0"/>
         <parent link="${chassis_link}"/>
@@ -61,5 +58,7 @@
       </joint>
       <joint name="front_${lr_prefix}_wheel_joint" type="fixed">
-        <origin xyz="0 0 0"
+        <origin xyz="${wheelbase / 2}
+                     ${lr_reflect * ((chassis_width - wheel_width) / 2)}
+                     ${elevacion_coche}"
                 rpy="0 0 0"/>
         <parent link="${lr_prefix}_steering_hinge"/>
@@ -70,10 +69,32 @@
       <xacro:wheel lr_prefix="${lr_prefix}" fr_prefix="front"/>
     </xacro:macro>
-    <!-- Description of how a rear wheel is connected to the chassis -->
+     <xacro:macro name="front_wheel_l" params="lr_prefix lr_reflect">
+      <link name="${lr_prefix}_steering_hinge"/>
+      <joint name="${lr_prefix}_steering_hinge_joint" type="revolute">
+        <origin xyz="0 0 0"
+                rpy="0 0 0"/>
+        <parent link="${chassis_link}"/>
+        <child link="${lr_prefix}_steering_hinge"/>
+        <axis xyz="0 0 1"/>
+        <limit lower="${-1*steering_limit}" upper="${steering_limit}" effort="10000000" velocity="1000000"/>
+      </joint>
+      <joint name="front_${lr_prefix}_wheel_joint" type="fixed">
+        <origin xyz="${wheelbase / 2}
+                     ${lr_reflect * ((chassis_width - wheel_width) / 2)}
+                     ${elevacion_coche}"
+                rpy="${2*degrees_90} 0 0"/>
+        <parent link="${lr_prefix}_steering_hinge"/>
+        <child link="${lr_prefix}_front_wheel"/>
+        <axis xyz="0 1 0"/>
+        <limit lower="0" upper="0" effort="10000000" velocity="1000000"/>
+      </joint>
+      <xacro:wheel lr_prefix="${lr_prefix}" fr_prefix="front"/>
+    </xacro:macro>
+    <!-- Description of how a rear wheel is connected to the ch-->
     <xacro:macro name="rear_wheel" params="lr_prefix lr_reflect">
-      <joint name="rear_${lr_prefix}_wheel_joint" type="fixed">
+      <joint name="rear_${lr_prefix}_wheel_joint" type="revolute">
         <origin xyz="${-1 * wheelbase / 2}
                      ${lr_reflect * ((chassis_width - wheel_width) / 2)}
-                     0"
+                     ${elevacion_coche}"
                 rpy="0 0 0"/>
         <parent link="${chassis_link}"/>
@@ -84,9 +105,21 @@
       <xacro:wheel lr_prefix="${lr_prefix}" fr_prefix="rear"/>
     </xacro:macro>
-    <!-- Add the wheels -->
-    <xacro:front_wheel lr_prefix="left" lr_reflect="1"/>
+    <xacro:macro name="rear_wheel_l" params="lr_prefix lr_reflect">
+      <joint name="rear_${lr_prefix}_wheel_joint" type="prismatic">
+        <origin xyz="${-1 * wheelbase / 2}
+                     ${lr_reflect * ((chassis_width - wheel_width) / 2)}
+                     ${elevacion_coche}"
+                rpy="${2*degrees_90} 0 0"/>
+        <parent link="${chassis_link}"/>
+        <child link="${lr_prefix}_rear_wheel"/>
+        <axis xyz="0 1 0"/>
+        <limit lower="0" upper="0" effort="10000000" velocity="1000000"/>
+      </joint>
+      <xacro:wheel lr_prefix="${lr_prefix}" fr_prefix="rear"/>
+    </xacro:macro>
+    <xacro:front_wheel_l lr_prefix="left" lr_reflect="1"/>
     <xacro:front_wheel lr_prefix="right" lr_reflect="-1"/>
-    <xacro:rear_wheel lr_prefix="left" lr_reflect="1" />
+    <xacro:rear_wheel_l lr_prefix="left" lr_reflect="1" />
     <xacro:rear_wheel lr_prefix="right" lr_reflect="-1" />
-  </xacro:macro>
+</xacro:macro>
 </robot>
